File: EMF.brd (EAGLE design)
At the start: 49.2 x 63.5 mm, 23 parts, among them X1 22-23-2021

Commit message: fixing stuff
Parts:
- C1: value .1uF -> 0.1uF
- C12, C16: value 100nF -> 0.1uF
Changed lines of the file:
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@@
 <elements>
 <element name="C.AMP" library="linear" library_urn="urn:adsk.eagle:library:262" package="SO08" package3d_urn="urn:adsk.eagle:package:16404/2" value="LM741D" x="33.02" y="46.99" rot="MR270"/>
-<element name="C1" library="SparkFun" package="0805" value=".1uF" x="35.56" y="45.212"/>
+<element name="C1" library="SparkFun" package="0805" value="0.1uF" x="35.56" y="45.212"/>
 <element name="C11" library="SparkFun" package="0805" value="10uF" x="22.86" y="63.373" rot="MR270"/>
-<element name="C12" library="SparkFun" package="0805" value="100nF" x="25.908" y="65.151" rot="MR90"/>
+<element name="C12" library="SparkFun" package="0805" value="0.1uF" x="25.908" y="65.151" rot="MR90"/>
 <element name="C15" library="SparkFun" package="0805" value="10uF" x="21.209" y="44.45" rot="R90"/>
-<element name="C16" library="SparkFun" package="0805" value="100nF" x="24.13" y="44.45" rot="R90"/>
+<element name="C16" library="SparkFun" package="0805" value="0.1uF" x="24.13" y="44.45" rot="R90"/>
 <element name="DIODE" library="Physoon" package="LILYPAD-WEARABLES_LED-1206" value="" x="5.334" y="64.389" rot="MR180"/>
 <element name="IC1" library="xmega-a4" package="QFP80P1200X1200X120-44N" value="" x="22.86" y="53.34" rot="R180"/>

Commit message: fix op-amp connections
Connections:
- net GND: now also C.AMP.3, V.AMP.3; no longer C.AMP.2, C1.2, R4.1
- net S2(VIN): now also C.AMP.2, C1.2, R4.1; no longer C.AMP.3, V.AMP.3
Routing:
- net S2(VIN): track 15.4 -> 14.0 mm
Changed lines of the file:
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@@
 <signal name="S2(VIN)">
 <contactref element="X1" pad="2"/>
-<contactref element="C.AMP" pad="3"/>
-<contactref element="V.AMP" pad="3"/>
-<wire x1="41.275" y1="47.371" x2="40.259" y2="46.355" width="0.4064" layer="16"/>
-<wire x1="40.259" y1="46.355" x2="35.62" y2="46.355" width="0.4064" layer="16"/>
-<wire x1="36.86729375" y1="53.3606" x2="36.2344" y2="53.3606" width="0.4064" layer="16"/>
-<wire x1="36.2344" y1="53.3606" x2="35.62" y2="53.975" width="0.4064" layer="16"/>
-<wire x1="41.275" y1="47.371" x2="41.275" y2="48.95289375" width="0.4064" layer="16"/>
-<wire x1="41.275" y1="48.95289375" x2="36.86729375" y2="53.3606" width="0.4064" layer="16"/>
+<contactref element="C.AMP" pad="2"/>
+<contactref element="C1" pad="2"/>
+<contactref element="R4" pad="1"/>
+<wire x1="36.51" y1="45.162" x2="36.46" y2="45.212" width="0.4064" layer="1"/>
+<wire x1="41.275" y1="47.371" x2="35.874" y2="47.371" width="0.4064" layer="16"/>
+<wire x1="35.874" y1="47.371" x2="35.62" y2="47.625" width="0.4064" layer="16"/>
+<wire x1="36.51" y1="43.434" x2="36.51" y2="45.162" width="0.4064" layer="1"/>
+<wire x1="41.275" y1="47.371" x2="37.338" y2="43.434" width="0.4064" layer="1"/>
+<wire x1="37.338" y1="43.434" x2="36.51" y2="43.434" width="0.4064" layer="1"/>
 </signal>
 <signal name="N$3">
@@
 <contactref element="JP4" pad="5"/>
 <contactref element="X1" pad="1"/>
-<contactref element="C.AMP" pad="2"/>
-<contactref element="C1" pad="2"/>
-<contactref element="R4" pad="1"/>
-<wire x1="36.51" y1="45.162" x2="36.46" y2="45.212" width="0.4064" layer="1"/>
 <polygon width="0.4064" layer="1">
 <vertex x="0" y="16.51"/>
@@
 <contactref element="MPU" pad="4"/>
 <contactref element="XB1" pad="10"/>
-<wire x1="4.699" y1="41.402" x2="16.94" y2="36.94" width="0" layer="19" extent="1-1"/>
+<contactref element="C.AMP" pad="3"/>
+<contactref element="V.AMP" pad="3"/>
 </signal>
 <signal name="V+">

Commit message: fix naming convention
Connections:
- net S2(VIN) renamed S1(VIN)
Changed lines of the file:
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@@
 </elements>
 <signals>
-<signal name="S2(VIN)">
+<signal name="S1(VIN)">
 <contactref element="X1" pad="2"/>
 <contactref element="C.AMP" pad="2"/>
