File: EFM.kicad_pcb (KiCad board)
At the start: 2 copper layers, 49.2 x 57 mm, 36 parts, among them J1 Openlog, J2 IMU, J3 Spheres, J4 AVR-PDI-6, M1 SHC_123_BATTERY_HOLDERCR-123-A, U1 TPS60400DBVR, U2 LM741, U3 LM741, U4 XCL206B, U5 ATxmega32A4U-AU

Commit message: Small updates
Routing:
- net Net-(C3-Pad1): track 10.1 -> 13.5 mm, vias 1 -> 2
- net /VOUT: track 17.4 -> 20.5 mm, vias 0 -> 1
Other:
- board text added: "C"
- board text added: "V"
Changed lines of the file:
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@@
   (general
     (thickness 1.6)
-    (drawings 9)
-    (tracks 219)
+    (drawings 11)
+    (tracks 227)
     (zones 0)
     (modules 36)
@@
       (xy -0.000753 4.598977) (xy 0.026181 4.598588)) (layer B.SilkS) (width 0.01))
   )
+  (gr_text V (at 226.5 67.4) (layer F.SilkS)
+    (effects (font (size 1.5 1.5) (thickness 0.3)) (justify mirror))
+  )
+  (gr_text C (at 230.1 67.35 180) (layer F.SilkS)
+    (effects (font (size 1.5 1.5) (thickness 0.3)) (justify mirror))
+  )
   (gr_text "EFM Rev 3.0" (at 203.15 70.2) (layer B.SilkS)
     (effects (font (size 1.5 1.5) (thickness 0.3)) (justify mirror))
@@
   (segment (start 231.6 63.8) (end 231.165 63.365) (width 0.25) (layer F.Cu) (net 4))
   (segment (start 231.6 65.4) (end 231.6 66.975) (width 0.25) (layer B.Cu) (net 4))
+  (via (at 229 67.4) (size 0.8) (drill 0.4) (layers F.Cu B.Cu) (net 4))
+  (segment (start 231.6 65.4) (end 231 65.4) (width 0.25) (layer F.Cu) (net 4))
+  (segment (start 231 65.4) (end 229 67.4) (width 0.25) (layer F.Cu) (net 4))
   (segment (start 233.2 63.2) (end 232.6 63.8) (width 0.25) (layer B.Cu) (net 5))
   (segment (start 240.6 63.2) (end 233.2 63.2) (width 0.25) (layer B.Cu) (net 5))
@@
   (segment (start 233.55 74.6) (end 233.55 73.8) (width 0.25) (layer F.Cu) (net 24))
   (segment (start 227.775 70.27) (end 228.8 70.27) (width 0.25) (layer F.Cu) (net 24))
-  (segment (start 224.27 70.27) (end 227.775 70.27) (width 0.25) (layer F.Cu) (net 24))
   (segment (start 221.2 67.2) (end 224.27 70.27) (width 0.25) (layer F.Cu) (net 24))
   (segment (start 221.2 66.2) (end 221.2 67.2) (width 0.25) (layer F.Cu) (net 24))
+  (via (at 227.65 67.45) (size 0.8) (drill 0.4) (layers F.Cu B.Cu) (net 24))
+  (segment (start 227.5 67.6) (end 227.65 67.45) (width 0.25) (layer F.Cu) (net 24))
+  (segment (start 227.5 69.67) (end 227.5 67.6) (width 0.25) (layer F.Cu) (net 24))
+  (segment (start 226.9 70.27) (end 227.5 69.67) (width 0.25) (layer F.Cu) (net 24))
+  (segment (start 226.9 70.27) (end 227.775 70.27) (width 0.25) (layer F.Cu) (net 24))
+  (segment (start 224.27 70.27) (end 226.9 70.27) (width 0.25) (layer F.Cu) (net 24))
   (segment (start 208.0375 45.725) (end 207.4 45.725) (width 0.25) (layer B.Cu) (net 31))
   (segment (start 208.3375 46.025) (end 208.0375 45.725) (width 0.25) (layer B.Cu) (net 31))
